Commit message: Clean up world / turtlebot spawning
- Pass the gazebo model path to the bookstore world launch file so it's
not hardcoded any more.
- Change spawning turtlebot to use spawn_entity.py now instead of
running shell commands.
- Add ability to set turtlebot initial pose
- Convert xacro files to urdf because it can't be done on the fly with
spawn_entity.py

File: simulation_ws/src/turtlebot3_description_reduced_mesh/urdf/turtlebot3_waffle.urdf (robot description, URDF)
Before this commit: robot turtlebot3_waffle, 13 links, 12 joints
Joints:
- joint camera_depth_joint: origin xyz=0.005 0.028 0.013 rpy=0 0 0 -> xyz=0.005 0.027999999999999997 0.013 rpy=0 0 0
